File: maame_carrier.kicad_sch (KiCad schematic)
At the start: 67 parts, among them J1 Kakute left pad strip: 2x9 ma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, J10 FS-iA10B iBUS servo lead (S +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, J11 TF-Luna pin order 1-6 (CFG ti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, J12 Spare FC I2C (5 V supply, sha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, J13 Payload servo power (+ -); se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, J17 Kakute spare: T3 RSSI 3V3(FC)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, J18 Pi SPI0, 3V3 logic, J20 VBAT OUT 6S fused (JST-XH 2-p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, J21 9V OUT from Kakute VTX 9V (JS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, J22 12V OUT 2A (JST-XH), J23 Kakute top pads G 5V Vi CAM: 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, J24 Kakute bottom pads Z- 5V G LE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, J25 Kakute JST 9V T1 R1 G: 1x4 ma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, J3 VBAT tap from ESC battery pad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, J6 Spare power: 5V_AUX G 5V_FC G, J7 Pi expansion: 3V3 logic ONLY, J8 TBS M10Q: order matches its p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, J9 SiK radio (UART4), U1 Pi Zero W socket: 2x20 female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, U2 TPS54360BDDAR 60V 3.5A buck, U3 TPS54360BDDAR 12V 2A buck

Commit message: Board named MaameDrone V1.0: silkscreen, title blocks (rev 1.0), notes; fab outputs renamed MaameDrone_V1.0_*
Other:
- note added: "MaameDrone V1.0 carrier board (rev 1.0)"
- note removed: "MAAME CARRIER BOARD rev A (draft, layout pending frame measurements)"
- title: Maame carrier board -> MaameDrone V1.0
Changed lines of the file:
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@@
 	(paper "A3")
 	(title_block
-		(title "Maame carrier board")
+		(title "MaameDrone V1.0")
 		(date "2026-10-27")
-		(rev "A-draft")
+		(rev "1.0")
 		(comment 1 "Base board under Kakute H7 V1.5 (ESC separate), Pi Zero W socket, peripheral headers")
 	)
@@
 		)
 	)
-	(text "MAAME CARRIER BOARD  rev A (draft, layout pending frame measurements)"
+	(text "MaameDrone V1.0 carrier board (rev 1.0)"
 		(exclude_from_sim no)
 		(at 20.32 243.84 0)

Commit message: Remove 12 V buck (U3, L2, D10, C9-C15, R12-R16, D11, J22) and 9 V output (J21); J25 pin 1 no net (9V DO NOT WIRE); F1 back to 2 A 1812 (C960026); re-routed, DRC/ERC 0 errors; fab regenerated
Parts:
- removed C10, C9: 2.2uF 100V X7R 1210 (12V VIN), Capacitor_SMD:C_1210_3225Metric, symbol maame_carrier:Capacitor
- removed C11: 100nF 50V 0603 (12V BOOT), Capacitor_SMD:C_0603_1608Metric, symbol maame_carrier:Capacitor
- removed C12: 15nF 50V 0603 (12V COMP), Capacitor_SMD:C_0603_1608Metric, symbol maame_carrier:Capacitor
- removed C13: 56pF 50V C0G 0603 (12V COMP), Capacitor_SMD:C_0603_1608Metric, symbol maame_carrier:Capacitor
- removed C14, C15: 22uF 25V X7R 1210 (12V OUT), Capacitor_SMD:C_1210_3225Metric, symbol maame_carrier:Capacitor
- removed D10: B560C 60V 5A Schottky SMC, Diode_SMD:D_SMC, symbol maame_carrier:Schottky
- removed D11: Green 0805: 12V_AUX on, LED_SMD:LED_0805_2012Metric_Pad1.15x1.40mm_HandSolder, symbol maame_carrier:LED
- removed J21: 9V OUT from Kakute VTX 9V (JST-XH), Connector_JST:JST_XH_B2B-XH-A_1x02_P2.50mm_Vertical, symbol maame_carrier:BEC_OUT
- removed J22: 12V OUT 2A (JST-XH), Connector_JST:JST_XH_B2B-XH-A_1x02_P2.50mm_Vertical, symbol maame_carrier:BEC_OUT
- removed L2: 22uH 5.9A Coilcraft XAL6060-223MEC, Inductor_SMD:L_Coilcraft_XAL6060-XXX, symbol maame_carrier:Inductor
- removed R12: 162k 1% 0603 (12V RT, 600 kHz), Resistor_SMD:R_0603_1608Metric, symbol maame_carrier:Resistor
- removed R13: 9.1k 1% 0603 (12V COMP), Resistor_SMD:R_0603_1608Metric, symbol maame_carrier:Resistor
- removed R14: 140k 1% 0603 (12V FB top), Resistor_SMD:R_0603_1608Metric, symbol maame_carrier:Resistor
- removed R15: 10k 1% 0603 (12V FB bottom), Resistor_SMD:R_0603_1608Metric, symbol maame_carrier:Resistor
- removed R16: 2.2k 0805 (12V LED), Resistor_SMD:R_0805_2012Metric_Pad1.20x1.40mm_HandSolder, symbol maame_carrier:Resistor
- removed U3: TPS54360BDDAR 12V 2A buck, Package_SO:TI_SO-PowerPAD-8_ThermalVias, symbol maame_carrier:TPS54360B
- F1: value PTC fuse 2920 30V 3A hold 6A trip (BSMD2920-300-30V, LCSC C7190311) -> PTC fuse 1812 30V 2A hold 4A trip (BSMD1812-200-30V, LCSC C960026); footprint Fuse:Fuse_2920_7451Metric -> Fuse:Fuse_1812_4532Metric_Pad1.30x3.40mm_HandSolder; LCSC C7190311 -> C960026
- J25: value Kakute JST 9V T1 R1 G: 1x4 male header (JLC THT) -> Kakute JST 9V(NC) T1 R1 G: 1x4 male header (JLC THT)
Connections:
- net 9V_FC: no longer names the net of J25.1
Other:
- note added: "11. No 12 V buck and no 9 V output (both removed for assembly cost). J25 pin 1 (Kakute 9V) has no net: DO NOT WIRE."
- note added: "8. Power: 6S Li-ion (18-25.2 V) from J3 tap -> F1 PTC (2 A hold, 4 A trip, 30 V) -> D9 SMBJ30A TVS (clamps surges to ~48 V, under U2 60 V max) -> U2 5 V buck (note 10) -> 5V_AUX. J20 VBAT OUT (JST-XH) takes VBAT before F1 through its own F2 (2 A). Battery: 6S Li-ion/LiPo only, 18-25.2 V (22.2 V nom). Full 3.5 A out at 18 V in draws ~1.1 A."
- note removed: "11. 12V_AUX: second TPS54360B, 12 V 2 A from VBAT_F. Values from TI SNVSB93 eqs 28-51: 600 kHz (162k), L 22 uH (Isat 5.9 A), Cout 2x22 uF 25 V, FB 140k/10k = 12.0 V, comp 9.1k + 15 nF, 56 pF. 9V_FC = Kakute VTX 9 V (J1 pad 30), current per Holybro spec (unconfirmed). F1 3 A hold: 5 V full (1.1 A) + 12 V full (1.5 A) at 18 V in = 2.6 A."
- note removed: "8. Power: 6S Li-ion (18-25.2 V) from J3 tap -> F1 PTC (3 A hold, 6 A trip, 30 V, 2920) -> D9 SMBJ30A TVS (clamps surges to ~48 V, under U2 60 V max) -> U2 5 V buck (note 10) -> 5V_AUX. J20 VBAT OUT (JST-XH) takes VBAT before F1 through its own F2 (2 A). Battery: 6S Li-ion/LiPo only, 18-25.2 V (22.2 V nom). Full 3.5 A out at 18 V in draws ~1.1 A."

Commit message: Pi mounts FACE DOWN (header on top of Pi, as on a Zero WH): U1 footprint mirrored along the header axis (pin 1 at the right end, SD right, USB/HDMI rear); Pi silkscreen redone; re-routed, DRC/ERC 0 errors; fab, renders and PDF regenerated
Parts:
- U1: footprint maame_carrier:Pi_Zero_Socketed_FaceUp_MountingHoles -> maame_carrier:Pi_Zero_Socketed_FaceDown_MountingHoles
Changed lines of the file:
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@@
 			)
 		)
-		(property "Footprint" "maame_carrier:Pi_Zero_Socketed_FaceUp_MountingHoles"
+		(property "Footprint" "maame_carrier:Pi_Zero_Socketed_FaceDown_MountingHoles"
 			(at 330.2 35.56 0)
 			(hide yes)

Commit message: JLC assembles SMD only: J1, J23-J25 and U1 Pi socket moved to hand-solder (excluded from BOM/CPL, still in 3D); 32 parts / 21 BOM lines; parts-to-buy list in ASSEMBLY_NOTES
Parts:
- J1, J23, J24, J25, U1: now left out of the parts list
Changed lines of the file:
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@@
 		(body_style 1)
 		(exclude_from_sim no)
-		(in_bom yes)
+		(in_bom no)
 		(on_board yes)
 		(in_pos_files yes)
@@
 		(body_style 1)
 		(exclude_from_sim no)
-		(in_bom yes)
+		(in_bom no)
 		(on_board yes)
 		(in_pos_files yes)
@@
 		(body_style 1)
 		(exclude_from_sim no)
-		(in_bom yes)
+		(in_bom no)
 		(on_board yes)
 		(in_pos_files yes)
@@
 		(body_style 1)
 		(exclude_from_sim no)
-		(in_bom yes)
+		(in_bom no)
 		(on_board yes)
 		(in_pos_files yes)
@@
 		(body_style 1)
 		(exclude_from_sim no)
-		(in_bom yes)
+		(in_bom no)
 		(on_board yes)
 		(in_pos_files yes)
